File: hardware/Schematics/IoT_Power_Meter_schematics.sch (KiCad schematic (older format))
At the start: 9 parts, among them SW1 SW_PUSH, U1 ESP-12, U2 AP1117T33, U3 FTDI

Commit message: fix
Parts:
- 10K2: symbol R -> Device:R
- C1: symbol Power_connector -> IoT_Power_Meter_schematics-rescue:Power_connector
- D1: symbol OLED -> IoT_Power_Meter_schematics-rescue:OLED
- S1: symbol LightSensor -> IoT_Power_Meter_schematics-rescue:LightSensor
- SD1: symbol MicroSD -> IoT_Power_Meter_schematics-rescue:MicroSD
- SW1: symbol SW_PUSH -> IoT_Power_Meter_schematics-rescue:SW_PUSH
- U1: symbol ESP-12 -> IoT_Power_Meter_schematics-rescue:ESP-12
- U2: symbol AP1117T33 -> IoT_Power_Meter_schematics-rescue:AP1117T33
- U3: symbol FTDI -> IoT_Power_Meter_schematics-rescue:FTDI
Changed lines of the file:
@@
-EESchema Schematic File Version 2
-LIBS:power
-LIBS:device
-LIBS:transistors
-LIBS:conn
-LIBS:linear
-LIBS:regul
-LIBS:74xx
-LIBS:cmos4000
-LIBS:adc-dac
-LIBS:memory
-LIBS:xilinx
-LIBS:microcontrollers
-LIBS:dsp
-LIBS:microchip
-LIBS:analog_switches
-LIBS:motorola
-LIBS:texas
-LIBS:intel
-LIBS:audio
-LIBS:interface
-LIBS:digital-audio
-LIBS:philips
-LIBS:display
-LIBS:cypress
-LIBS:siliconi
-LIBS:opto
-LIBS:atmel
-LIBS:contrib
-LIBS:valves
-LIBS:MyLibrary
-LIBS:ESP8266
-LIBS:IoT_Power_Meter_schematics-cache
-EELAYER 25 0
+EESchema Schematic File Version 4
+EELAYER 30 0
 EELAYER END
 $Descr A4 11693 8268
@@
 $EndDescr
 $Comp
-L ESP-12 U1
+L IoT_Power_Meter_schematics-rescue:ESP-12 U1
 U 1 1 56744217
 P 4550 3800
@@
 $EndComp
 $Comp
-L GND #PWR01
+L power:GND #PWR01
 U 1 1 5674428B
 P 4550 4700
@@
 $EndComp
 $Comp
-L VCC #PWR02
+L power:VCC #PWR02
 U 1 1 567442BA
 P 4550 2900
@@
 $EndComp
 $Comp
-L GND #PWR03
+L power:GND #PWR03
 U 1 1 567443DB
 P 5450 4100
@@
 $EndComp
 $Comp
-L R 10K2
+L Device:R 10K2
 U 1 1 567456FA
 P 6400 4500
@@
 $EndComp
 $Comp
-L VCC #PWR04
+L power:VCC #PWR04
 U 1 1 56745878
 P 8650 3400
@@
 $EndComp
 $Comp
-L GND #PWR05
+L power:GND #PWR05
 U 1 1 56745885
 P 8650 4300
@@
 $EndComp
 $Comp
-L OLED D1
+L IoT_Power_Meter_schematics-rescue:OLED D1
 U 1 1 56747219
 P 8650 3850
@@
 $EndComp
 $Comp
-L MicroSD SD1
+L IoT_Power_Meter_schematics-rescue:MicroSD SD1
 U 1 1 567474F3
 P 4550 5850
@@
 MOSI
 $Comp
-L VCC #PWR06
+L power:VCC #PWR06
 U 1 1 5674776B
 P 4550 5400
@@
 $EndComp
 $Comp
-L GND #PWR07
+L power:GND #PWR07
 U 1 1 5674777B
 P 4550 6300
@@
 $EndComp
 $Comp
-L LightSensor S1
+L IoT_Power_Meter_schematics-rescue:LightSensor S1
 U 1 1 567479DB
 P 8650 2450
@@
 $EndComp
 $Comp
-L GND #PWR08
+L power:GND #PWR08
 U 1 1 56747A6E
 P 8650 2850
@@
 $EndComp
 $Comp
-L VCC #PWR09
+L power:VCC #PWR09
 U 1 1 56747A91
 P 8650 2050
@@
 $EndComp
 $Comp
-L FTDI U3
+L IoT_Power_Meter_schematics-rescue:FTDI U3
 U 1 1 56747C70
 P 6400 2450
@@
 $EndComp
 $Comp
-L GND #PWR010
+L power:GND #PWR010
 U 1 1 56747ED7
 P 6400 2850
@@
 $EndComp
 $Comp
-L SW_PUSH SW1
+L IoT_Power_Meter_schematics-rescue:SW_PUSH SW1
 U 1 1 56748014
 P 6400 4950
@@
 $EndComp
 $Comp
-L GND #PWR011
+L power:GND #PWR011
 U 1 1 56748102
 P 6400 5250
@@
 $EndComp
 $Comp
-L VCC #PWR012
+L power:VCC #PWR012
 U 1 1 5674812B
 P 6400 4350
@@
 NoConn ~ 3650 3600
 $Comp
-L AP1117T33 U2
+L IoT_Power_Meter_schematics-rescue:AP1117T33 U2
 U 1 1 5676A1C5
 P 3850 1600
@@
 $EndComp
 $Comp
-L GND #PWR013
+L power:GND #PWR013
 U 1 1 5676A2BC
 P 3850 1900
@@
 $EndComp
 $Comp
-L VCC #PWR014
+L power:VCC #PWR014
 U 1 1 5676A372
 P 4300 1450
@@
 $EndComp
 $Comp
-L +5V #PWR015
+L power:+5V #PWR015
 U 1 1 5676A3A1
 P 3400 1450
@@
 RX
 $Comp
-L +5V #PWR016
+L power:+5V #PWR016
 U 1 1 5679B6EF
 P 6400 2050
@@
 The ESP-12 and ESP-12E have GPIO4/5\nswapped, otherwise they are stricly\nthe same, this can be changed in software
 $Comp
-L Power_connector C1
+L IoT_Power_Meter_schematics-rescue:Power_connector C1
 U 1 1 56F85C43
 P 2050 1600
@@
 $EndComp
 $Comp
-L GND #PWR018
+L power:GND #PWR018
 U 1 1 56F85D63
 P 2050 2000
@@
 $EndComp
 $Comp
-L +5V #PWR?
+L power:+5V #PWR?
 U 1 1 56F863C3
 P 2050 1200

Commit message: fix
Parts:
- C1: symbol IoT_Power_Meter_schematics-rescue:Power_connector -> IoT_Power_Meter_schematics-rescue:Power_connector-IoT_Power_Meter_schematics-rescue
- D1: symbol IoT_Power_Meter_schematics-rescue:OLED -> IoT_Power_Meter_schematics-rescue:OLED-IoT_Power_Meter_schematics-rescue
- S1: symbol IoT_Power_Meter_schematics-rescue:LightSensor -> IoT_Power_Meter_schematics-rescue:LightSensor-IoT_Power_Meter_schematics-rescue
- SD1: symbol IoT_Power_Meter_schematics-rescue:MicroSD -> IoT_Power_Meter_schematics-rescue:MicroSD-IoT_Power_Meter_schematics-rescue
- SW1: symbol IoT_Power_Meter_schematics-rescue:SW_PUSH -> IoT_Power_Meter_schematics-rescue:SW_PUSH-IoT_Power_Meter_schematics-rescue
- U1: symbol IoT_Power_Meter_schematics-rescue:ESP-12 -> IoT_Power_Meter_schematics-rescue:ESP-12-IoT_Power_Meter_schematics-rescue
- U2: symbol IoT_Power_Meter_schematics-rescue:AP1117T33 -> IoT_Power_Meter_schematics-rescue:AP1117T33-IoT_Power_Meter_schematics-rescue
- U3: symbol IoT_Power_Meter_schematics-rescue:FTDI -> IoT_Power_Meter_schematics-rescue:FTDI-IoT_Power_Meter_schematics-rescue
Changed lines of the file:
@@
 $EndDescr
 $Comp
-L IoT_Power_Meter_schematics-rescue:ESP-12 U1
+L IoT_Power_Meter_schematics-rescue:ESP-12-IoT_Power_Meter_schematics-rescue U1
 U 1 1 56744217
 P 4550 3800
@@
 $EndComp
 $Comp
-L IoT_Power_Meter_schematics-rescue:OLED D1
+L IoT_Power_Meter_schematics-rescue:OLED-IoT_Power_Meter_schematics-rescue D1
 U 1 1 56747219
 P 8650 3850
@@
 $EndComp
 $Comp
-L IoT_Power_Meter_schematics-rescue:MicroSD SD1
+L IoT_Power_Meter_schematics-rescue:MicroSD-IoT_Power_Meter_schematics-rescue SD1
 U 1 1 567474F3
 P 4550 5850
@@
 $EndComp
 $Comp
-L IoT_Power_Meter_schematics-rescue:LightSensor S1
+L IoT_Power_Meter_schematics-rescue:LightSensor-IoT_Power_Meter_schematics-rescue S1
 U 1 1 567479DB
 P 8650 2450
@@
 $EndComp
 $Comp
-L IoT_Power_Meter_schematics-rescue:FTDI U3
+L IoT_Power_Meter_schematics-rescue:FTDI-IoT_Power_Meter_schematics-rescue U3
 U 1 1 56747C70
 P 6400 2450
@@
 $EndComp
 $Comp
-L IoT_Power_Meter_schematics-rescue:SW_PUSH SW1
+L IoT_Power_Meter_schematics-rescue:SW_PUSH-IoT_Power_Meter_schematics-rescue SW1
 U 1 1 56748014
 P 6400 4950
@@
 NoConn ~ 3650 3600
 $Comp
-L IoT_Power_Meter_schematics-rescue:AP1117T33 U2
+L IoT_Power_Meter_schematics-rescue:AP1117T33-IoT_Power_Meter_schematics-rescue U2
 U 1 1 5676A1C5
 P 3850 1600
@@
 The ESP-12 and ESP-12E have GPIO4/5\nswapped, otherwise they are stricly\nthe same, this can be changed in software
 $Comp
-L IoT_Power_Meter_schematics-rescue:Power_connector C1
+L IoT_Power_Meter_schematics-rescue:Power_connector-IoT_Power_Meter_schematics-rescue C1
 U 1 1 56F85C43
 P 2050 1600
